File: schematic/bumblebee/layerboards/psu_board.brd (EAGLE design)
At the start: 100 x 80 mm, 17 parts, among them Q1 IRF9530, Q2 IRF540, Q3 IRF9530, Q4 IRF540, Q5 IRF9530, Q6 IRF540, Q7 IRF9530, Q8 IRF540

Commit message: Squashed commit of the following:
commit bbe75f2ba636e86ea759fc0c795d406c2297ca99
Author: Kirs67 <kirilel200267@gmail.com>
Date:   Mon Jan 7 01:16:28 2019 +0300

    Исправлена INA

commit 84fcf59dae87e7c5b0b953ea137079167e3747d4
Author: Kirs67 <kirilel200267@gmail.com>
Date:   Mon Jan 7 00:40:04 2019 +0300

    Добавлена схема выключения

commit 4c991518a2578b81abe136c16c09ad2ddfd2125b
Author: Kirs67 <kirilel200267@gmail.com>
Date:   Sun Jan 6 23:47:41 2019 +0300

    Добавлена поддержка USB type C
Parts:
- added D1, D2, D3, D4: 1N4446, diode:DO35-10
- added DC4: (no value), dc-dc-converter:NME
- added Q9: IRF540, transistor-power:TO220BV
- added U$5: PCB_USB_CDS_5, USB_pcb_connectors:USB_TYPE_C_DS_5
- added U$6, U$7: CHARGER, bluepill:CHARGER
Connections:
- new net N$18: D1.C, Q9.G
- new net N$19: DC4.2, U$5.A4, U$5.A9, U$5.B4, U$5.B9
- new net N$2: D1.A, D2.C, D3.C, D4.A
- new net N$20: G1.-, U$7.B-
- new net N$21: G2.+, U$7.B+
- new net N$24: DC4.1, DC4.3, Q9.S, U$5.A1, U$5.A12, U$5.B1, U$5.B12, U$7.P-
- new net TCK: U$5.A11, U$5.B11
- new net TDI_USB: U$5.A2, U$5.B2
- new net TDO_USB: U$5.A3, U$5.B3
- new net TMS: U$5.A10, U$5.B10
- new net USB_CC1: U$1.A4, U$5.A5
- new net USB_CC2: U$1.A5, U$5.B5
- new net USB_DMINUS: U$5.A7, U$5.B7
- new net USB_DPLUS: U$5.A6, U$5.B6
- new net USB_SBU1: D3.A, U$5.A8
- new net USB_SBU2: D2.A, U$5.B8
- net 5V_CONTINUOUS: now also D4.C
- net 7.4V: now also DC4.4, U$7.P+; no longer G2.+
- net GND: now also Q9.D; no longer G1.-
- net N$17: now also U$7.BALANCE
