File: schematic/bumblebee/layerboards/psu_board.brd (EAGLE design)
At the start: 85 x 100 mm, 50 parts, among them Q1 IRF9530, Q10 IRF9530, Q2 IRF9530, Q3 IRF9530, Q5 IRF9530, Q7 IRF9530, T1 2N7002E, T2 2N7002E, T3 2N7002E, T4 2N7002E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

Commit message: Правки по PSU
Parts:
- removed KEY_1, KEY_2: (no value), pinhead:1X01
- added P1: B3B-EH-A, con-jst-eh:B3B-EH-A
Connections:
- net GND: now also P1.1, P1.3
- net KEY_1: no longer KEY_1.1
- net KEY_2: no longer KEY_2.1
- net N$22: now also P1.2
Routing:
- net N$22: track 9.61 -> 26.9 mm
- net KEY_2: track 149.6 -> 145.7 mm
- net KEY_1: track 15.6 -> 12.7 mm
Changed lines of the file:
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@@
 <attribute name="VALUE" x="42.66" y="5.445" size="1.27" layer="27"/>
-</element>
-<element name="KEY_1" library="pinhead" library_urn="urn:adsk.eagle:library:325" package="1X01" package3d_urn="urn:adsk.eagle:package:22485/2" value="" x="14.84" y="15.72" smashed="yes">
-<attribute name="NAME" x="13.4938" y="17.5488" size="1.27" layer="25" ratio="10"/>
-<attribute name="VALUE" x="13.57" y="12.545" size="1.27" layer="27"/>
-</element>
-<element name="KEY_2" library="pinhead" library_urn="urn:adsk.eagle:library:325" package="1X01" package3d_urn="urn:adsk.eagle:package:22485/2" value="" x="14.82" y="18.62" smashed="yes">
-<attribute name="NAME" x="13.4738" y="20.4488" size="1.27" layer="25" ratio="10"/>
-<attribute name="VALUE" x="13.55" y="15.445" size="1.27" layer="27"/>
 </element>
 <element name="LED1" library="led" library_urn="urn:adsk.eagle:library:259" package="LED5MM" package3d_urn="urn:adsk.eagle:package:15799/2" value="" x="79.74" y="55.47" smashed="yes" rot="R90">
@@
 <attribute name="NAME" x="54.953" y="7.759" size="1.016" layer="25" ratio="18"/>
 <attribute name="VALUE" x="54.953" y="1.917" size="1.016" layer="27" ratio="10"/>
+</element>
+<element name="P1" library="con-jst-eh" package="B3B-EH-A" value="B3B-EH-A" x="17.8" y="5.8" smashed="yes" rot="R180">
+<attribute name="NAME" x="21.737" y="3.641" size="1.016" layer="25" ratio="18" rot="R180"/>
+<attribute name="VALUE" x="21.737" y="9.483" size="1.016" layer="27" ratio="10" rot="R180"/>
 </element>
 </elements>
@@
 <vertex x="0" y="0"/>
 </polygon>
+<contactref element="P1" pad="1"/>
+<contactref element="P1" pad="3"/>
+<wire x1="66.75" y1="78.23" x2="69.72" y2="83.9" width="0" layer="19" extent="1-1"/>
+<wire x1="69.52" y1="62.43" x2="66.75" y2="78.23" width="0" layer="19" extent="1-1"/>
+<wire x1="66.75" y1="55.52" x2="69.52" y2="62.43" width="0" layer="19" extent="1-1"/>
+<wire x1="79.74" y1="56.74" x2="69.52" y2="62.43" width="0" layer="19" extent="1-1"/>
+<wire x1="81.07" y1="65.21" x2="79.74" y2="56.74" width="0" layer="19" extent="1-1"/>
+<wire x1="69.52" y1="38.86" x2="66.75" y2="55.52" width="0" layer="19" extent="1-1"/>
+<wire x1="66.89" y1="32.52" x2="69.52" y2="38.86" width="0" layer="19" extent="1-1"/>
+<wire x1="69.41" y1="15.18" x2="66.89" y2="32.52" width="0" layer="19" extent="1-1"/>
+<wire x1="66.89" y1="9.23" x2="69.41" y2="15.18" width="0" layer="19" extent="1-1"/>
+<wire x1="48.91" y1="16.61" x2="66.89" y2="9.23" width="0" layer="19" extent="1-1"/>
+<wire x1="43.93" y1="8.62" x2="48.91" y2="16.61" width="0" layer="19" extent="1-1"/>
+<wire x1="30.92" y1="13.17" x2="43.93" y2="8.62" width="0" layer="19" extent="1-1"/>
+<wire x1="20.01" y1="11.12" x2="30.92" y2="13.17" width="0" layer="19" extent="1-1"/>
+<wire x1="22.67" y1="29.57" x2="30.92" y2="13.17" width="0" layer="19" extent="1-1"/>
+<wire x1="18.13" y1="48.78" x2="22.67" y2="29.57" width="0" layer="19" extent="1-1"/>
+<wire x1="29.56" y1="48.78" x2="18.13" y2="48.78" width="0" layer="19" extent="1-1"/>
+<wire x1="6.3" y1="48.22" x2="18.13" y2="48.78" width="0" layer="19" extent="1-1"/>
+<wire x1="46.3" y1="48.22" x2="29.56" y2="48.78" width="0" layer="19" extent="1-1"/>
+<wire x1="15.3" y1="5.8" x2="20.01" y2="11.12" width="0" layer="19" extent="1-1"/>
+<wire x1="20.3" y1="5.8" x2="15.3" y2="5.8" width="0" layer="19" extent="1-1"/>
+<wire x1="46.41" y1="71.01" x2="66.75" y2="78.23" width="0" layer="19" extent="1-1"/>
+<wire x1="6.41" y1="71.01" x2="6.3" y2="48.22" width="0" layer="19" extent="1-1"/>
+<wire x1="6.43" y1="80.32" x2="6.41" y2="71.01" width="0" layer="19" extent="1-1"/>
+<wire x1="6.23" y1="94.01" x2="6.43" y2="80.32" width="0" layer="19" extent="1-1"/>
+<wire x1="46.23" y1="94.01" x2="46.41" y2="71.01" width="0" layer="19" extent="1-1"/>
+<wire x1="33.37" y1="94.5" x2="46.23" y2="94.01" width="0" layer="19" extent="1-1"/>
+<wire x1="33.37" y1="91.96" x2="33.37" y2="94.5" width="0" layer="19" extent="1-1"/>
 </signal>
 <signal name="5V_CONTINUOUS">
@@
 </signal>
 <signal name="KEY_1">
-<contactref element="KEY_1" pad="1"/>
 <contactref element="BAT+" pad="1"/>
 <contactref element="Q2" pad="S"/>
 <contactref element="R10" pad="P$1"/>
-<wire x1="14.83" y1="11.12" x2="14.83" y2="15.71" width="1.5" layer="1"/>
-<wire x1="14.83" y1="15.71" x2="14.84" y2="15.72" width="1.5" layer="1"/>
-<wire x1="14.84" y1="15.72" x2="20.16" y2="15.72" width="1.5" layer="1"/>
 <wire x1="20.16" y1="15.72" x2="20.19" y2="15.69" width="1.5" layer="1"/>
 <wire x1="20.19" y1="15.69" x2="20.19" y2="19.74" width="1.5" layer="1"/>
 <wire x1="20.19" y1="19.74" x2="21.31" y2="20.86" width="1.5" layer="1"/>
+<wire x1="20.19" y1="15.69" x2="14.83" y2="11.12" width="1.5" layer="1"/>
 </signal>
 <signal name="KEY_2">
 <contactref element="Q1" pad="S"/>
-<contactref element="KEY_2" pad="1"/>
 <contactref element="U$4" pad="IN+"/>
 <contactref element="U$5" pad="IN+"/>
@@
 <wire x1="36.39" y1="15.78" x2="36.39" y2="19.42" width="1" layer="1"/>
 <wire x1="36.39" y1="19.42" x2="37.93" y2="20.96" width="1" layer="1"/>
-<wire x1="14.82" y1="18.62" x2="19.584" y2="23.384" width="1.5" layer="1"/>
 <wire x1="23.85" y1="21.75" x2="23.85" y2="20.86" width="1.5" layer="1"/>
-<wire x1="19.584" y1="23.384" x2="22.216" y2="23.384" width="1.5" layer="1"/>
-<wire x1="22.216" y1="23.384" x2="23.85" y2="21.75" width="1.5" layer="1"/>
-<wire x1="14.82" y1="18.62" x2="6.3" y2="27.14" width="1.5" layer="1"/>
+<wire x1="23.85" y1="21.75" x2="22.216" y2="23.384" width="1.5" layer="1"/>
 <wire x1="6.3" y1="27.14" x2="6.3" y2="30.22" width="1.5" layer="1"/>
 <wire x1="6.3" y1="30.22" x2="6.3" y2="44.9" width="1.5" layer="1"/>
@@
 <wire x1="36.4" y1="6" x2="46.25730625" y2="6" width="0.8" layer="1"/>
 <wire x1="46.25730625" y1="6" x2="51.28730625" y2="11.03" width="0.8" layer="1"/>
+<wire x1="10.056" y1="23.384" x2="6.3" y2="27.14" width="1.5" layer="1"/>
+<wire x1="22.216" y1="23.384" x2="10.056" y2="23.384" width="1.5" layer="1"/>
 </signal>
 <signal name="N$22">
@@
 <wire x1="27.81" y1="15.69" x2="27.81" y2="13.13" width="0.6" layer="1"/>
 <wire x1="27.81" y1="13.13" x2="28.72" y2="12.22" width="0.6" layer="1"/>
+<wire x1="24.15" y1="18.62" x2="26.39" y2="20.86" width="0.3" layer="16"/>
+<contactref element="P1" pad="2"/>
+<wire x1="27.81" y1="15.69" x2="17.92" y2="5.8" width="0.3" layer="16"/>
+<wire x1="17.92" y1="5.8" x2="17.8" y2="5.8" width="0.3" layer="16"/>
 </signal>
 <signal name="KILLSWITCH">
