File: schematic/bumblebee/layerboards/ccu_board.sch (EAGLE design)
At the start: 0 parts

Commit message: RC платок аппарата
Parts:
- added P1: B4B-EH-A, con-jst-eh:B4B-EH-A
- added R1: (no value), ngspice-simulation:R
- added U$1: PX4FLOW, bluepill:PX4FLOW
- added U$2: CAM_BIG, bluepill:CAM_BIG
- added U$3: CAM, bluepill:CAM
- added U$4: MCP2551, MCP2551:MCP2551
Connections:
- new net 5V_CCU: P1.1, U$1.5V, U$2.5V, U$3.5V, U$4.VDD
- new net GND: P1.4, R1.2, U$1.GND, U$2.GND, U$3.GND, U$4.VSS
- new net N$1: U$1.USART3_RX, U$2.TX
- new net N$2: U$1.USART3_TX, U$2.RX
- new net N$3: U$1.USART2_RX, U$3.TX
- new net N$4: U$1.USART2_TX, U$3.RX
- new net N$5: U$1.USB_D+, U$4.TXD
- new net N$6: U$1.USB_D-, U$4.RXD
- new net N$7: R1.1, U$4.RS
- new net N$8: P1.2, U$4.CANH
- new net N$9: P1.3, U$4.CANL
