File: schematic/bumblebee/layerboards/psu_board.sch (EAGLE design)
At the start: 26 parts, among them Q1 IRF9530, Q2 IRF540, Q3 IRF9530, Q4 IRF540, Q5 IRF9530, Q6 IRF540, Q7 IRF9530, Q8 IRF540

Commit message: Squashed commit of the following:
commit bbe75f2ba636e86ea759fc0c795d406c2297ca99
Author: Kirs67 <kirilel200267@gmail.com>
Date:   Mon Jan 7 01:16:28 2019 +0300

    Исправлена INA

commit 84fcf59dae87e7c5b0b953ea137079167e3747d4
Author: Kirs67 <kirilel200267@gmail.com>
Date:   Mon Jan 7 00:40:04 2019 +0300

    Добавлена схема выключения

commit 4c991518a2578b81abe136c16c09ad2ddfd2125b
Author: Kirs67 <kirilel200267@gmail.com>
Date:   Sun Jan 6 23:47:41 2019 +0300

    Добавлена поддержка USB type C
Parts:
- added D1, D2, D3, D4: 1N4446, diode:1N4446
- added DC4: (no value), dc-dc-converter:NME
- added Q9: IRF540, transistor-power:IRF540
- added R10: 82k, ngspice-simulation:R
- added R11: 8.2k, ngspice-simulation:R
- added U$5: PCB_USB_CDS_5, USB_pcb_connectors:PCB_USB_CDS_5
- added U$6, U$7: CHARGER, bluepill:CHARGER
- added U$8, U$9: INA, bluepill:INA
Connections:
- removed net 7.4V: DC1.+VIN, DC2.+VIN, DC3.+VIN, G2.+, Q1.S, R1.2
- removed net PCTRL_PCU: Q8.G, R8.1
- new net KEY_MINUS: R11.2
- new net KEY_PLUS: DC1.+VIN, DC2.+VIN, DC3.+VIN, DC4.+VOUT, Q1.S, R1.2, U$7.P+
- new net N$18: D1.C, Q9.G, R10.2, R11.1
- new net N$19: DC4.+VIN, U$5.A4, U$5.A9, U$5.B4, U$5.B9
- new net N$2: D1.A, D2.C, D3.C, D4.A
- new net N$20: G1.-, U$7.B-
- new net N$21: G2.+, U$7.B+
- new net N$24: DC4.-VIN, DC4.-VOUT, Q9.S, R10.1, U$5.A1, U$5.A12, U$5.B1, U$5.B12, U$7.P-
- new net TCK: U$5.A11, U$5.B11
- new net TDI_USB: U$5.A2, U$5.B2
- new net TDO_USB: U$5.A3, U$5.B3
- new net TMS: U$5.A10, U$5.B10
- new net USB_CC1: U$1.PA4, U$5.A5
- new net USB_CC2: U$1.PA5, U$5.B5
- new net USB_DMINUS: U$5.A7, U$5.B7
- new net USB_DPLUS: U$5.A6, U$5.B6
- new net USB_SBU1: D3.A, U$5.A8
- new net USB_SBU2: D2.A, U$5.B8
- net 5V_CCU: now also U$9.VIN-; no longer U$2.VIN-_0
- net 5V_CONTINUOUS: now also D4.C, U$8.VCC, U$9.VCC
- net 5V_ICU: now also U$2.VIN-; no longer U$3.VIN-_0
- net 5V_SCU: now also U$8.VIN-; no longer U$3.VIN-_1
- net GND: now also Q9.D, U$8.GND, U$9.GND; no longer G1.-
- net HEATER: now also U$3.VIN-; no longer U$2.VIN-_1
- net N$10: now also U$8.VIN+; no longer U$3.VIN+_1
- net N$11: now also U$2.VIN+; no longer U$3.VIN+_0
- net N$12: now also U$1.PB11, U$2.SDA, U$3.SDA, U$8.SDA, U$9.SDA; no longer U$1.PB10, U$2.SCL, U$3.SCL
- net N$13: now also U$1.PB10, U$2.SCL, U$3.SCL, U$8.SCL, U$9.SCL; no longer U$1.PB11, U$2.SDA, U$3.SDA
- net N$17: now also U$7.BALANCE
- net N$8: now also U$3.VIN+; no longer U$2.VIN+_1
- net N$9: now also U$9.VIN+; no longer U$2.VIN+_0
- net PCTRL_ICU: now also Q8.G, R8.1
Other:
- moved on the sheet: DC1, DC2, DC3, G1, G2, Q1, Q2, Q3, Q4, Q5, Q6, Q7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

Commit message: RC платок аппарата
Parts:
- removed U$6: CHARGER, bluepill:CHARGER
- added P1, P2: B5B-EH-A, con-jst-eh:B5B-EH-A
- added P3: B3B-EH-A, con-jst-eh:B3B-EH-A
- added P4: B4B-EH-A, con-jst-eh:B4B-EH-A
- added R12, R13: 26k, ngspice-simulation:R
Connections:
- removed net HEATER: U$3.VIN-
- removed net TCK: U$5.A11, U$5.B11
- removed net TDI_USB: U$5.A2, U$5.B2
- removed net TDO_USB: U$5.A3, U$5.B3
- removed net TMS: U$5.A10, U$5.B10
- new net 7.4V: P2.2, U$3.VIN-
- new net SWCLK_0: U$1.SWCLK, U$5.A3
- new net SWCLK_1: P3.2, U$5.A10
- new net SWCLK_2: P4.3, U$5.B3
- new net SWCLK_3: P4.1, U$5.B10
- new net SWDIO_0: U$1.SWDIO, U$5.A2
- new net SWDIO_1: P3.1, U$5.A11
- new net SWDIO_2: P4.4, U$5.B2
- new net SWDIO_3: P4.2, U$5.B11
- net 5V_CCU: now also P1.4
- net 5V_ICU: now also P2.1
- net 5V_SCU: now also P1.5
- net CANH: now also P1.3, P2.3
- net CANL: now also P1.2, P2.4
- net GND: now also P1.1, R12.1, R13.1
- net USB_CC1: now also R13.2
- net USB_CC2: now also R12.2
