File: schematic/bumblebee/layerboards/psu_board.sch (EAGLE design)
At the start: 44 parts, among them P1 B5B-EH-A, P2 B5B-EH-A, P3 B3B-EH-A, P4 B4B-EH-A, Q1 IRF9530, Q2 IRF540, Q3 IRF9530, Q4 IRF540, Q5 IRF9530, Q6 IRF540, Q7 IRF9530, Q8 IRF540, Q9 IRF540

Commit message: Начата работа над платами Design-block iridium ICU МК Начал переделывать схему ICU
Connections:
- net GND: now also P2.5
Changed lines of the file:
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@@
 <?xml version="1.0" encoding="utf-8"?>
 <!DOCTYPE eagle SYSTEM "eagle.dtd">
-<eagle version="9.2.2">
+<eagle version="9.3.0">
 <drawing>
 <settings>
@@
 <pinref part="GND14" gate="1" pin="GND"/>
 <wire x1="-5.08" y1="-96.52" x2="-5.08" y2="-104.14" width="0.1524" layer="91"/>
+<pinref part="P2" gate="G$1" pin="5"/>
+<wire x1="20.32" y1="-96.52" x2="-5.08" y2="-96.52" width="0.1524" layer="91"/>
+<junction x="-5.08" y="-96.52"/>
 </segment>
 </net>

Commit message: Скоро будут готовы ICU, SCU и CCU. Остались последние проверки
Parts:
- removed D1, D2, D3, D4: 1N4446, diode:1N4446
- added P5: B3B-EH-A, con-jst-eh:B3B-EH-A
Connections:
- removed net N$18: D1.C, Q9.G, R10.2, R11.1
- removed net N$2: D1.A, D2.C, D3.C, D4.A
- new net KEY_PCU: Q9.G, R10.2, R11.1, U$1.PA9
- net 5V_CONTINUOUS: no longer D4.C
- net GND: now also P5.3
- net KEY_MINUS: now also P5.1
- net KEY_PLUS: now also P5.2
- net USB_SBU1: no longer D3.A
- net USB_SBU2: no longer D2.A
Changed lines of the file:
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@@
 <part name="R10" library="ngspice-simulation" library_urn="urn:adsk.eagle:library:527439" deviceset="R" device="" value="82k"/>
 <part name="R11" library="ngspice-simulation" library_urn="urn:adsk.eagle:library:527439" deviceset="R" device="" value="8.2k"/>
-<part name="D1" library="diode" library_urn="urn:adsk.eagle:library:210" deviceset="1N4446" device="" package3d_urn="urn:adsk.eagle:package:43344/2"/>
-<part name="D2" library="diode" library_urn="urn:adsk.eagle:library:210" deviceset="1N4446" device="" package3d_urn="urn:adsk.eagle:package:43344/2"/>
-<part name="D3" library="diode" library_urn="urn:adsk.eagle:library:210" deviceset="1N4446" device="" package3d_urn="urn:adsk.eagle:package:43344/2"/>
-<part name="D4" library="diode" library_urn="urn:adsk.eagle:library:210" deviceset="1N4446" device="" package3d_urn="urn:adsk.eagle:package:43344/2"/>
 <part name="U$2" library="bluepill" deviceset="INA" device=""/>
 <part name="GND7" library="supply1" library_urn="urn:adsk.eagle:library:371" deviceset="GND" device=""/>
@@
 <part name="P3" library="con-jst-eh" deviceset="B3B-EH-A" device=""/>
 <part name="P4" library="con-jst-eh" deviceset="B4B-EH-A" device=""/>
+<part name="P5" library="con-jst-eh" deviceset="B3B-EH-A" device=""/>
+<part name="GND15" library="supply1" library_urn="urn:adsk.eagle:library:371" deviceset="GND" device=""/>
 </parts>
 <sheets>
@@
 <attribute name="VALUE" x="-115.57" y="5.08" size="1.778" layer="96" rot="R90"/>
 </instance>
-<instance part="D1" gate="1" x="-129.54" y="2.54" smashed="yes">
-<attribute name="NAME" x="-127" y="3.0226" size="1.778" layer="95"/>
-</instance>
-<instance part="D2" gate="1" x="-139.7" y="-5.08" smashed="yes">
-<attribute name="NAME" x="-137.16" y="-7.1374" size="1.778" layer="95"/>
-</instance>
-<instance part="D3" gate="1" x="-139.7" y="10.16" smashed="yes">
-<attribute name="NAME" x="-137.16" y="10.6426" size="1.778" layer="95"/>
-</instance>
-<instance part="D4" gate="1" x="-134.62" y="2.54" smashed="yes" rot="R180">
-<attribute name="NAME" x="-137.16" y="2.0574" size="1.778" layer="95" rot="R180"/>
-</instance>
 <instance part="U$2" gate="G$1" x="35.56" y="-45.72" smashed="yes"/>
 <instance part="GND7" gate="1" x="17.78" y="-50.8" smashed="yes">
@@
 <attribute name="NAME" x="-115.57" y="-97.155" size="1.778" layer="95" rot="R180"/>
 <attribute name="VALUE" x="-115.57" y="-81.28" size="1.778" layer="95" rot="R180"/>
+</instance>
+<instance part="P5" gate="G$1" x="-63.5" y="-109.22" smashed="yes">
+<attribute name="NAME" x="-64.77" y="-103.505" size="1.778" layer="95"/>
+<attribute name="VALUE" x="-64.77" y="-116.84" size="1.778" layer="95"/>
+</instance>
+<instance part="GND15" gate="1" x="-88.9" y="-116.84" smashed="yes">
+<attribute name="VALUE" x="-91.44" y="-119.38" size="1.778" layer="96"/>
 </instance>
 </instances>
@@
 <wire x1="20.32" y1="-96.52" x2="-5.08" y2="-96.52" width="0.1524" layer="91"/>
 <junction x="-5.08" y="-96.52"/>
+</segment>
+<segment>
+<pinref part="P5" gate="G$1" pin="3"/>
+<wire x1="-68.58" y1="-111.76" x2="-88.9" y2="-111.76" width="0.1524" layer="91"/>
+<wire x1="-88.9" y1="-111.76" x2="-88.9" y2="-114.3" width="0.1524" layer="91"/>
+<pinref part="GND15" gate="1" pin="GND"/>
 </segment>
 </net>
@@
 <label x="-88.9" y="20.32" size="1.778" layer="95"/>
 </segment>
+<segment>
+<pinref part="P5" gate="G$1" pin="2"/>
+<wire x1="-68.58" y1="-109.22" x2="-88.9" y2="-109.22" width="0.1524" layer="91"/>
+<label x="-83.82" y="-109.22" size="1.778" layer="95"/>
+</segment>
 </net>
 <net name="5V_CONTINUOUS" class="0">
@@
 </segment>
 <segment>
-<pinref part="D4" gate="1" pin="C"/>
-<wire x1="-137.16" y1="2.54" x2="-157.48" y2="2.54" width="0.1524" layer="91"/>
-<label x="-157.48" y="2.54" size="1.778" layer="95"/>
-</segment>
-<segment>
 <pinref part="U$2" gate="G$1" pin="VCC"/>
 <wire x1="22.86" y1="-50.8" x2="22.86" y2="-53.34" width="0.1524" layer="91"/>
@@
 <wire x1="-114.3" y1="-33.02" x2="-101.6" y2="-33.02" width="0.1524" layer="91"/>
 <label x="-114.3" y="-33.02" size="1.778" layer="95"/>
-</segment>
-<segment>
-<pinref part="D2" gate="1" pin="A"/>
-<wire x1="-142.24" y1="-5.08" x2="-157.48" y2="-5.08" width="0.1524" layer="91"/>
-<label x="-157.48" y="-5.08" size="1.778" layer="95"/>
 </segment>
 </net>
@@
 <label x="-154.94" y="-40.64" size="1.778" layer="95"/>
 </segment>
-<segment>
-<pinref part="D3" gate="1" pin="A"/>
-<wire x1="-142.24" y1="10.16" x2="-157.48" y2="10.16" width="0.1524" layer="91"/>
-<label x="-157.48" y="10.16" size="1.778" layer="95"/>
-</segment>
-</net>
-<net name="N$18" class="0">
+</net>
+<net name="KEY_PCU" class="0">
 <segment>
 <pinref part="R10" gate="G$1" pin="2"/>
@@
 <pinref part="R11" gate="G$1" pin="1"/>
 <junction x="-119.38" y="2.54"/>
-<pinref part="D1" gate="1" pin="C"/>
-<wire x1="-127" y1="2.54" x2="-119.38" y2="2.54" width="0.1524" layer="91"/>
-</segment>
-</net>
-<net name="N$2" class="0">
-<segment>
-<pinref part="D2" gate="1" pin="C"/>
-<pinref part="D1" gate="1" pin="A"/>
-<wire x1="-137.16" y1="-5.08" x2="-132.08" y2="-2.54" width="0.1524" layer="91"/>
-<wire x1="-132.08" y1="-2.54" x2="-132.08" y2="2.54" width="0.1524" layer="91"/>
-<pinref part="D3" gate="1" pin="C"/>
-<wire x1="-137.16" y1="10.16" x2="-132.08" y2="7.62" width="0.1524" layer="91"/>
-<wire x1="-132.08" y1="7.62" x2="-132.08" y2="2.54" width="0.1524" layer="91"/>
-<junction x="-132.08" y="2.54"/>
-<pinref part="D4" gate="1" pin="A"/>
+<wire x1="-119.38" y1="2.54" x2="-139.7" y2="2.54" width="0.1524" layer="91"/>
+<label x="-137.16" y="2.54" size="1.778" layer="95"/>
+</segment>
+<segment>
+<pinref part="U$1" gate="G$1" pin="PA9"/>
+<wire x1="119.38" y1="-20.32" x2="132.08" y2="-20.32" width="0.1524" layer="91"/>
+<label x="121.92" y="-20.32" size="1.778" layer="95"/>
 </segment>
 </net>
@@
 <label x="-88.9" y="25.4" size="1.778" layer="95"/>
 </segment>
-</net>
+<segment>
+<pinref part="P5" gate="G$1" pin="1"/>
+<wire x1="-68.58" y1="-106.68" x2="-88.9" y2="-106.68" width="0.1524" layer="91"/>
+<label x="-83.82" y="-106.68" size="1.778" layer="95"/>
+</segment>
+</net>

Commit message: Сделана платка PCU, осталось развести. Добавлена ещё одна либа для игла
Parts:
- removed DC1, DC2, DC3, DC4: (no value), dc-dc-converter:NME
- removed G1, G2: SL-160AA/PT, battery:SL-160AA/PT
- removed P3, P5: B3B-EH-A, con-jst-eh:B3B-EH-A
- removed Q4, Q6, Q8, Q9: IRF540, transistor-power:IRF540
- added BAT+, BAT-, KEY_1, KEY_2: (no value), pinhead:PINHD-1X1
- added DEBUG_FROM_ICU, KEY_TO_OUT: B3B-EH-A, con-jst-eh:B3B-EH-A
- added DEBUG_TO_OUT: B8B-EH-A, con-jst-eh:B8B-EH-A
- added LED1: (no value), led:LED5MM
- added Q10: IRF9530, transistor-power:IRF9530
- added R14, R15, R16, R17, R18: 10k, SparkFun-Resistors:RESISTORAXIAL-0.3
- added T1, T2, T3, T4, T5, T6: 2N7002E, nxp_60:2N7002E
- added U$6: CAN, bluepill:CAN
- Q2: value IRF540 -> IRF9530; device transistor-power:IRF540 -> transistor-power:IRF9530
- R1, R2, R3, R4, R5, R6, R7, R8: device ngspice-simulation:R -> SparkFun-Resistors:RESISTORAXIAL-0.3
- R10: value 82k -> 10k; device ngspice-simulation:R -> SparkFun-Resistors:RESISTORAXIAL-0.3
- R11: value 8.2k -> 10k; device ngspice-simulation:R -> SparkFun-Resistors:RESISTORAXIAL-0.3
- R12, R13: value 26k -> 10k; device ngspice-simulation:R -> SparkFun-Resistors:RESISTORAXIAL-0.3
- R9: value (none) -> 150; device ngspice-simulation:R -> SparkFun-Resistors:RESISTORAXIAL-0.3
- U$4: value MCP2551 -> DCDC; device MCP2551:MCP2551 -> bluepill:DCDC
- U$5: value PCB_USB_CDS_5 -> DCDC; device USB_pcb_connectors:PCB_USB_CDS_5 -> bluepill:DCDC
- U$7: value CHARGER -> DCDC; device bluepill:CHARGER -> bluepill:DCDC
- renumbered P1 to TO_SCU, P2 to TO_ICU, P4 to DEBUG_FROM_SCU
Connections:
- removed net KEY_PCU: Q9.G, R10.2, R11.1, U$1.PA9
- removed net N$24: DC4.-VIN, DC4.-VOUT, Q9.S, R10.1, U$5.A1, U$5.A12, U$5.B1, U$5.B12, U$7.P-
- removed net USB_CC1: R13.2, U$1.PA4, U$5.A5
- removed net USB_CC2: R12.2, U$1.PA5, U$5.B5
- removed net USB_DMINUS: U$5.A7, U$5.B7
- removed net USB_DPLUS: U$5.A6, U$5.B6
- removed net USB_SBU1: U$5.A8
- removed net USB_SBU2: U$5.B8
- new net 3V3: U$1.3V3, U$2.VCC, U$3.VCC, U$8.VCC, U$9.VCC
- new net HEATER_PLUS: Q10.D
- new net KEY_1: BAT+.1, KEY_1.1, Q2.S, R10.1
- new net KEY_2: KEY_2.1, Q1.S, Q2.D, R3.1, U$4.IN+, U$5.IN+, U$7.IN+
- new net KILLSWITCH: R11.2, T6.G, U$1.PA9
- new net N$18: R15.1, U$1.PA1
- new net N$2: U$1.PA11, U$6.CRX
- new net N$22: Q2.G, R10.2, T6.D
- new net PCTRL_AMP: R18.2, R4.2, T2.G
- net 5V_CONTINUOUS: now also R11.1, R13.1, R2.1, R4.1, R5.1, R6.1, R8.1, R9.1, U$4.OUT+; no longer DC1.+VOUT, R2.2, R3.2, R4.2, R6.2, R8.2, U$2.VCC, U$3.VCC, U$4.VDD, U$8.VCC, U$9.VCC
- net CANH: now also U$6.CANH; no longer U$4.CANH
- net CANL: now also U$6.CANL; no longer U$4.CANL
- net GND: now also BAT-.1, KEY_TO_OUT.3, LED1.C, T1.S, T2.S, T3.S, T4.S, T5.S, T6.S, U$4.IN-, U$4.OUT-, U$5.IN-, U$5.OUT-, U$7.IN-, U$7.OUT-; no longer DC1.-VIN, DC1.-VOUT, DC2.-VIN, DC2.-VOUT, DC3.-VIN, DC3.-VOUT, P5.3, Q2.S, Q4.S, Q6.S, Q8.S, Q9.D, R12.1, R13.1, R9.2, U$4.VSS
- net KEY_MINUS: now also KEY_TO_OUT.1; no longer P5.1, R11.2
- net KEY_PLUS: now also KEY_TO_OUT.2, Q10.S, R1.1; no longer DC1.+VIN, DC2.+VIN, DC3.+VIN, DC4.+VOUT, P5.2, Q1.S, R1.2, U$7.P+
- net N$1: now also R3.2, T2.D; no longer Q2.D, R1.1
- net N$14: now also U$6.CTX; no longer U$4.TXD
- net N$15: now also LED1.A, R9.2; no longer U$1.PA11, U$4.RXD
- net N$16: now also Q10.G, R1.2, T1.D; no longer R9.1, U$4.RS
- net N$17: now also R14.1, U$1.PA0; no longer G1.+, G2.-, U$7.BALANCE
- net N$19: now also R16.1, U$1.PA2; no longer DC4.+VIN, U$5.A4, U$5.A9, U$5.B4, U$5.B9
- net N$20: now also R17.1, U$1.PA3; no longer G1.-, U$7.B-
- net N$21: now also R18.1, U$1.PA4; no longer G2.+, U$7.B+
- net N$3: now also R7.2, T4.D; no longer Q6.D, R5.1
- net N$4: now also R12.2, T5.D; no longer Q8.D, R7.1
- net N$5: now also R7.1, U$5.OUT+; no longer DC2.+VOUT, R5.2
- net N$6: now also R5.2, T3.D; no longer Q4.D, R3.1
- net N$7: now also R12.1, U$7.OUT+; no longer DC3.+VOUT, R7.2
- net PCTRL_CCU: now also R14.2, R6.2, T3.G; no longer Q4.G, R4.1, U$1.PA0
- net PCTRL_HEATER: now also R17.2, R2.2, T1.G; no longer Q2.G, R2.1, U$1.PA3
- net PCTRL_ICU: now also R13.2, R16.2, T5.G; no longer Q8.G, R8.1, U$1.PA2
- net PCTRL_SCU: now also R15.2, R8.2, T4.G; no longer Q6.G, R6.1, U$1.PA1
- net SWCLK_0: now also DEBUG_TO_OUT.1; no longer U$5.A3
- net SWCLK_1: now also DEBUG_FROM_ICU.2, DEBUG_TO_OUT.3; no longer P3.2, U$5.A10
- net SWCLK_2: now also DEBUG_TO_OUT.5; no longer U$5.B3
- net SWCLK_3: now also DEBUG_TO_OUT.7; no longer U$5.B10
- net SWDIO_0: now also DEBUG_TO_OUT.2; no longer U$5.A2
- net SWDIO_1: now also DEBUG_FROM_ICU.1, DEBUG_TO_OUT.4; no longer P3.1, U$5.A11
- net SWDIO_2: now also DEBUG_TO_OUT.6; no longer U$5.B2
- net SWDIO_3: now also DEBUG_TO_OUT.8; no longer U$5.B11

Commit message: Finally finished with PCU. Pls check it
Parts:
- removed DEBUG_FROM_ICU, KEY_TO_OUT: B3B-EH-A, con-jst-eh:B3B-EH-A
- added HEATER_7.4V, HEATER_GND: (no value), pinhead:PINHD-1X1
- DEBUG_TO_OUT: value B8B-EH-A -> B6B-EH-A; device con-jst-eh:B8B-EH-A -> con-jst-eh:B6B-EH-A
Connections:
- removed net HEATER_PLUS: Q10.D
- removed net KEY_MINUS: KEY_TO_OUT.1
- removed net KEY_PLUS: KEY_TO_OUT.2, Q10.S, R1.1
- removed net SWCLK_1: DEBUG_FROM_ICU.2, DEBUG_TO_OUT.3
- removed net SWDIO_1: DEBUG_FROM_ICU.1, DEBUG_TO_OUT.4
- new net HEATER_7.4V: HEATER_7.4V.1, Q10.D
- net 3V3: now also U$6.3V3
- net GND: now also HEATER_GND.1, U$6.GND; no longer KEY_TO_OUT.3
- net KEY_2: now also Q10.S, R1.1
- net SWCLK_2: now also DEBUG_TO_OUT.4; no longer DEBUG_TO_OUT.5
- net SWCLK_3: now also DEBUG_TO_OUT.6; no longer DEBUG_TO_OUT.7
- net SWDIO_2: now also DEBUG_TO_OUT.3; no longer DEBUG_TO_OUT.6
- net SWDIO_3: now also DEBUG_TO_OUT.5; no longer DEBUG_TO_OUT.8

Commit message: Правки по PSU
Parts:
- removed KEY_1, KEY_2: (no value), pinhead:PINHD-1X1
- added P1: B3B-EH-A, con-jst-eh:B3B-EH-A
Connections:
- net GND: now also P1.1, P1.3
- net KEY_1: no longer KEY_1.1
- net KEY_2: no longer KEY_2.1
- net N$22: now also P1.2
Other:
- moved on the sheet: R11, T6
Changed lines of the file:
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@@
 <part name="GND3" library="supply1" library_urn="urn:adsk.eagle:library:371" deviceset="GND" device=""/>
 <part name="BAT+" library="pinhead" library_urn="urn:adsk.eagle:library:325" deviceset="PINHD-1X1" device="" package3d_urn="urn:adsk.eagle:package:22485/2"/>
-<part name="KEY_1" library="pinhead" library_urn="urn:adsk.eagle:library:325" deviceset="PINHD-1X1" device="" package3d_urn="urn:adsk.eagle:package:22485/2"/>
-<part name="KEY_2" library="pinhead" library_urn="urn:adsk.eagle:library:325" deviceset="PINHD-1X1" device="" package3d_urn="urn:adsk.eagle:package:22485/2"/>
 <part name="Q2" library="transistor-power" library_urn="urn:adsk.eagle:library:400" deviceset="IRF9530" device="" package3d_urn="urn:adsk.eagle:package:29484/3"/>
 <part name="GND13" library="supply1" library_urn="urn:adsk.eagle:library:371" deviceset="GND" device=""/>
@@
 <part name="DEBUG_TO_OUT" library="con-jst-eh" deviceset="B6B-EH-A" device=""/>
 <part name="GND16" library="supply1" library_urn="urn:adsk.eagle:library:371" deviceset="GND" device=""/>
+<part name="GND17" library="supply1" library_urn="urn:adsk.eagle:library:371" deviceset="GND" device=""/>
+<part name="P1" library="con-jst-eh" deviceset="B3B-EH-A" device=""/>
+<part name="GND18" library="supply1" library_urn="urn:adsk.eagle:library:371" deviceset="GND" device=""/>
 </parts>
 <sheets>
@@
 <attribute name="VALUE" x="-147.32" y="-54.61" size="1.778" layer="96" rot="R270"/>
 </instance>
-<instance part="KEY_1" gate="G$1" x="-152.4" y="-12.7" smashed="yes" rot="R90">
-<attribute name="NAME" x="-155.575" y="-19.05" size="1.778" layer="95" rot="R90"/>
-<attribute name="VALUE" x="-147.32" y="-19.05" size="1.778" layer="96" rot="R90"/>
-</instance>
-<instance part="KEY_2" gate="G$1" x="-142.24" y="-40.64" smashed="yes" rot="R270">
-<attribute name="NAME" x="-139.065" y="-34.29" size="1.778" layer="95" rot="R270"/>
-<attribute name="VALUE" x="-147.32" y="-34.29" size="1.778" layer="96" rot="R270"/>
-</instance>
 <instance part="Q2" gate="G$1" x="-177.8" y="-25.4" smashed="yes">
 <attribute name="NAME" x="-172.72" y="-22.86" size="1.778" layer="95"/>
 <attribute name="VALUE" x="-172.72" y="-25.4" size="1.778" layer="96"/>
 </instance>
-<instance part="GND13" gate="1" x="-182.88" y="-40.64" smashed="yes">
-<attribute name="VALUE" x="-185.42" y="-43.18" size="1.778" layer="96"/>
-</instance>
-<instance part="T6" gate="G$1" x="-185.42" y="-33.02" smashed="yes">
-<attribute name="VALUE" x="-179.07" y="-35.56" size="1.778" layer="96" font="vector"/>
-<attribute name="NAME" x="-179.07" y="-33.02" size="1.778" layer="95" font="vector"/>
+<instance part="GND13" gate="1" x="-182.88" y="-58.42" smashed="yes">
+<attribute name="VALUE" x="-185.42" y="-60.96" size="1.778" layer="96"/>
+</instance>
+<instance part="T6" gate="G$1" x="-185.42" y="-50.8" smashed="yes">
+<attribute name="VALUE" x="-179.07" y="-53.34" size="1.778" layer="96" font="vector"/>
+<attribute name="NAME" x="-179.07" y="-50.8" size="1.778" layer="95" font="vector"/>
 </instance>
 <instance part="U$4" gate="G$1" x="-91.44" y="25.4" smashed="yes">
@@
 <attribute name="VALUE" x="-184.404" y="-22.86" size="1.778" layer="96" font="vector" rot="R270" align="top-center"/>
 </instance>
-<instance part="R11" gate="G$1" x="-190.5" y="-30.48" smashed="yes" rot="R270">
-<attribute name="NAME" x="-188.976" y="-30.48" size="1.778" layer="95" font="vector" rot="R270" align="bottom-center"/>
-<attribute name="VALUE" x="-192.024" y="-30.48" size="1.778" layer="96" font="vector" rot="R270" align="top-center"/>
+<instance part="R11" gate="G$1" x="-190.5" y="-48.26" smashed="yes" rot="R270">
+<attribute name="NAME" x="-188.976" y="-48.26" size="1.778" layer="95" font="vector" rot="R270" align="bottom-center"/>
+<attribute name="VALUE" x="-192.024" y="-48.26" size="1.778" layer="96" font="vector" rot="R270" align="top-center"/>
 </instance>
 <instance part="R1" gate="G$1" x="2.54" y="68.58" smashed="yes" rot="R270">
@@
 <instance part="GND16" gate="1" x="99.06" y="-73.66" smashed="yes" rot="R90">
 <attribute name="VALUE" x="101.6" y="-76.2" size="1.778" layer="96" rot="R90"/>
+</instance>
+<instance part="GND17" gate="1" x="-223.52" y="-38.1" smashed="yes">
+<attribute name="VALUE" x="-226.06" y="-40.64" size="1.778" layer="96"/>
+</instance>
+<instance part="P1" gate="G$1" x="-200.66" y="-25.4" smashed="yes" rot="R90">
+<attribute name="NAME" x="-206.375" y="-26.67" size="1.778" layer="95" rot="R90"/>
+<attribute name="VALUE" x="-193.04" y="-26.67" size="1.778" layer="95" rot="R90"/>
+</instance>
+<instance part="GND18" gate="1" x="-190.5" y="-30.48" smashed="yes">
+<attribute name="VALUE" x="-193.04" y="-33.02" size="1.778" layer="96"/>
 </instance>
 </instances>
@@
 <wire x1="93.98" y1="-73.66" x2="96.52" y2="-73.66" width="0.1524" layer="91"/>
 <pinref part="GND16" gate="1" pin="GND"/>
+</segment>
+<segment>
+<wire x1="-203.2" y1="-33.02" x2="-223.52" y2="-33.02" width="0.1524" layer="91"/>
+<wire x1="-223.52" y1="-33.02" x2="-223.52" y2="-35.56" width="0.1524" layer="91"/>
+<pinref part="GND17" gate="1" pin="GND"/>
+<pinref part="P1" gate="G$1" pin="1"/>
+<wire x1="-203.2" y1="-33.02" x2="-203.2" y2="-30.48" width="0.1524" layer="91"/>
+</segment>
+<segment>
+<pinref part="P1" gate="G$1" pin="3"/>
+<wire x1="-198.12" y1="-30.48" x2="-195.58" y2="-30.48" width="0.1524" layer="91"/>
+<wire x1="-195.58" y1="-30.48" x2="-193.04" y2="-27.94" width="0.1524" layer="91"/>
+<wire x1="-193.04" y1="-27.94" x2="-190.5" y2="-27.94" width="0.1524" layer="91"/>
+<pinref part="GND18" gate="1" pin="GND"/>
 </segment>
 </net>
@@
 </segment>
 <segment>
-<wire x1="-190.5" y1="-25.4" x2="-210.82" y2="-25.4" width="0.1524" layer="91"/>
-<label x="-210.82" y="-25.4" size="1.778" layer="95"/>
+<wire x1="-190.5" y1="-43.18" x2="-210.82" y2="-43.18" width="0.1524" layer="91"/>
+<label x="-210.82" y="-43.18" size="1.778" layer="95"/>
 <pinref part="R11" gate="G$1" pin="1"/>
 </segment>
@@
 <net name="KEY_1" class="0">
 <segment>
-<label x="-154.94" y="-17.78" size="1.778" layer="95" rot="R270"/>
-<wire x1="-147.32" y1="-30.48" x2="-152.4" y2="-25.4" width="0.1524" layer="91"/>
-<wire x1="-152.4" y1="-25.4" x2="-152.4" y2="-15.24" width="0.1524" layer="91"/>
-<pinref part="KEY_1" gate="G$1" pin="1"/>
 <pinref part="BAT+" gate="G$1" pin="1"/>
 <wire x1="-142.24" y1="-58.42" x2="-142.24" y2="-50.8" width="0.1524" layer="91"/>
 <wire x1="-142.24" y1="-50.8" x2="-147.32" y2="-45.72" width="0.1524" layer="91"/>
 <wire x1="-147.32" y1="-45.72" x2="-147.32" y2="-30.48" width="0.1524" layer="91"/>
-</segment>
-<segment>
+<pinref part="R10" gate="G$1" pin="1"/>
 <pinref part="Q2" gate="G$1" pin="S"/>
 <wire x1="-175.26" y1="-20.32" x2="-175.26" y2="-17.78" width="0.1524" layer="91"/>
 <wire x1="-175.26" y1="-17.78" x2="-182.88" y2="-17.78" width="0.1524" layer="91"/>
-<wire x1="-175.26" y1="-17.78" x2="-162.56" y2="-17.78" width="0.1524" layer="91"/>
 <junction x="-175.26" y="-17.78"/>
+<wire x1="-175.26" y1="-17.78" x2="-152.4" y2="-17.78" width="0.1524" layer="91"/>
+<label x="-154.94" y="-17.78" size="1.778" layer="95" rot="R270"/>
 <label x="-170.18" y="-17.78" size="1.778" layer="95"/>
 <label x="-170.18" y="-17.78" size="1.778" layer="95"/>
-<pinref part="R10" gate="G$1" pin="1"/>
+<wire x1="-152.4" y1="-17.78" x2="-152.4" y2="-25.4" width="0.1524" layer="91"/>
+<wire x1="-152.4" y1="-25.4" x2="-147.32" y2="-30.48" width="0.1524" layer="91"/>
 </segment>
 </net>
@@
 <wire x1="-147.32" y1="-12.7" x2="-137.16" y2="-12.7" width="0.1524" layer="91"/>
 <wire x1="-147.32" y1="-12.7" x2="-147.32" y2="-25.4" width="0.1524" layer="91"/>
-<wire x1="-147.32" y1="-25.4" x2="-142.24" y2="-30.48" width="0.1524" layer="91"/>
-<wire x1="-142.24" y1="-30.48" x2="-142.24" y2="-38.1" width="0.1524" layer="91"/>
 <label x="-144.78" y="-25.4" size="1.778" layer="95" rot="R90"/>
-<pinref part="KEY_2" gate="G$1" pin="1"/>
 <pinref part="U$4" gate="G$1" pin="IN+"/>
 <wire x1="-119.38" y1="38.1" x2="-137.16" y2="38.1" width="0.1524" layer="91"/>
@@
 <pinref part="R3" gate="G$1" pin="1"/>
 <junction x="2.54" y="45.72"/>
-</segment>
-<segment>
 <pinref part="Q2" gate="G$1" pin="D"/>
-<wire x1="-162.56" y1="-30.48" x2="-175.26" y2="-30.48" width="0.1524" layer="91"/>
+<wire x1="-152.4" y1="-30.48" x2="-175.26" y2="-30.48" width="0.1524" layer="91"/>
 <label x="-170.18" y="-30.48" size="1.778" layer="95"/>
+<wire x1="-147.32" y1="-25.4" x2="-152.4" y2="-30.48" width="0.1524" layer="91"/>
 </segment>
 <segment>
@@
 <pinref part="R10" gate="G$1" pin="2"/>
 <junction x="-182.88" y="-27.94"/>
+<wire x1="-182.88" y1="-45.72" x2="-182.88" y2="-33.02" width="0.1524" layer="91"/>
+<junction x="-182.88" y="-45.72"/>
+<wire x1="-182.88" y1="-33.02" x2="-182.88" y2="-27.94" width="0.1524" layer="91"/>
+<junction x="-182.88" y="-33.02"/>
+<wire x1="-182.88" y1="-33.02" x2="-200.66" y2="-33.02" width="0.1524" layer="91"/>
+<pinref part="P1" gate="G$1" pin="2"/>
+<wire x1="-200.66" y1="-33.02" x2="-200.66" y2="-30.48" width="0.1524" layer="91"/>
 </segment>
 </net>
 <net name="KILLSWITCH" class="0">
 <segment>
-<wire x1="-187.96" y1="-35.56" x2="-190.5" y2="-35.56" width="0.1524" layer="91"/>
+<wire x1="-187.96" y1="-53.34" x2="-190.5" y2="-53.34" width="0.1524" layer="91"/>
 <pinref part="T6" gate="G$1" pin="G"/>
-<label x="-210.82" y="-35.56" size="1.778" layer="95"/>
+<label x="-210.82" y="-53.34" size="1.778" layer="95"/>
 <pinref part="R11" gate="G$1" pin="2"/>
-<wire x1="-190.5" y1="-35.56" x2="-210.82" y2="-35.56" width="0.1524" layer="91"/>
-<junction x="-190.5" y="-35.56"/>
-</segment>
-<segment>
+<wire x1="-190.5" y1="-53.34" x2="-210.82" y2="-53.34" width="0.1524" layer="91"/>
+<junction x="-190.5" y="-53.34"/>
+</segment>
+<segment>
