File: schematic/bumblebee/layerboards/icu_board.brd (EAGLE design)
At the start: 160 x 100 mm, 6 parts, among them P1 B5B-EH-A

Commit message: Готовая плата ICU. Стоит посмотреть ещё раз и проверить
Parts:
- removed U$2: MCP2551, MCP2551:SOIC-8
- added 10K, 10K1, 10K2: 10K, rcl:0204/7
- added ANT1, GPS1: MMCX-P-P-X-ST-TH1, MMCX-P-P-X-ST-TH1:MMCX-P-P-X-ST-TH1
- added ANT_IN, GPS_OUT: U.FL-R-SMT(01), U.FL-R-SMT_01_:HRS_U.FL-R-SMT(01)
- added C1: (no value), rcl:E3,5-8
- added C2: (no value), capacitor-wima:C2.5-2
- added JP1, JP2: (no value), pinhead:1X01
- added MK: 332-02, con-garry:332-02
- added U$4: ICU, bluepill:ICU
- added U$5: CAN, bluepill:CAN
- added USER_PORT1: SAMTEC-CLP-110-02-X-DJ, SAMTEC-CLP-110-02-X-D:SAMTEC-CLP-110-02-X-D
- GPS: value (none) -> 332-02; device pinhead:1X04 -> con-garry:332-02
- IRIDIUM: value (none) -> 332-02; device pinhead:2X10 -> con-garry:332-02
- U$1: value BLUEPILLTHEONLYONE -> GPS; device bluepill:BLUEPIL -> bluepill:GPS
- moved P1 82.4 mm to (75.5, 89.2), turned to 90 degrees
- moved GPS 72.5 mm to (16.4, 45.3), turned to 270 degrees
- moved U$3 46.5 mm to (21.2, 22.1), flipped to the bottom, turned to 270 degrees
- moved U$1 43.4 mm to (21.8, 22.8), turned to 270 degrees
- moved IRIDIUM 32.0 mm to (57.3, 46.3), turned to 90 degrees
Connections:
- removed net N$14: U$1.B12, U$3.P$19
- removed net N$19: U$1.C14, U$3.P$14
- new net DF_CTS: USER_PORT1.11
- new net DF_DCD: USER_PORT1.9
- new net DF_DSR: USER_PORT1.10
- new net DF_RI: U$4.PC9, USER_PORT1.12
- new net DF_S_RX: IRIDIUM.1, U$4.PB7, USER_PORT1.7
- new net DF_S_TX: IRIDIUM.2, U$4.PB6, USER_PORT1.6
- new net NETWORK_AVAILABLE: U$4.PE7, USER_PORT1.19
- new net ON_OFF: 10K.2, U$4.PB4, USER_PORT1.5
- new net PD8=TX: GPS.1, U$1.RX, U$4.PD8
- new net PD9=RX: GPS.2, U$1.TX, U$4.PD9
- new net RESERVED_1: USER_PORT1.16
- new net RESERVED_2\: USER_PORT1.17
- new net SUPPLY_OUT: USER_PORT1.20
- net 3.3V: now also 10K.1, 10K1.1, 10K2.1, U$4.3V3_0, U$5.3V3; no longer U$1.3V3_0, U$1.3V3_1, U$1.3V3_2
- net 5V_ICU: now also C1.+, C2.2, U$1.UCC, USER_PORT1.1, USER_PORT1.2; no longer GPS.4, IRIDIUM.1, IRIDIUM.2, U$2.VDD
- net 7.4V: now also JP1.1
- net GND: now also ANT1.2, ANT1.3, ANT1.4, ANT1.5, ANT_IN.1, ANT_IN.2, C1.-, C2.1, GPS1.2, GPS1.3, GPS1.4, GPS1.5, GPS_OUT.1, GPS_OUT.2, JP2.1, MK.1, U$1.GND, U$5.GND, USER_PORT1.13, USER_PORT1.14, USER_PORT1.15, USER_PORT1.18, USER_PORT1.3, USER_PORT1.4, USER_PORT1.8; no longer GPS.1, IRIDIUM.15, IRIDIUM.18, IRIDIUM.3, IRIDIUM.4, IRIDIUM.8, U$2.VSS
- net N$1: now also P1.3, U$5.CANH; no longer IRIDIUM.5, U$1.A4
- net N$10: now also U$4.PD1, U$5.CRX; no longer U$1.A12, U$2.RXD
- net N$11: now also 10K2.2, MK.2, U$4.PD7; no longer U$2.RS
- net N$12: now also U$3.P$13, U$4.PD15; no longer P1.3, U$2.CANH
- net N$13: now also U$3.P$8, U$4.PD13; no longer P1.2, U$2.CANL
- net N$15: now also U$3.P$17, U$4.PB15; no longer U$1.B13, U$3.P$18
- net N$16: now also U$3.P$16, U$4.PB14; no longer U$1.B15, U$3.P$17
- net N$17: now also U$3.P$14, U$4.PE12; no longer U$1.B14, U$3.P$16
- net N$18: now also 10K1.2, U$4.PE14; no longer U$1.C13
- net N$2: now also U$3.P$19, U$4.PB12; no longer GPS.3, U$1.B10
- net N$3: now also P1.2, U$5.CANL; no longer IRIDIUM.11, U$1.A1
- net N$4: now also ANT1.1, ANT_IN.3; no longer IRIDIUM.13, U$1.A0
- net N$5: now also GPS1.1, GPS_OUT.3; no longer IRIDIUM.7, U$1.A2
- net N$6: now also U$3.P$6, U$4.PE15; no longer IRIDIUM.6, U$1.A3
- net N$7: now also U$3.P$7, U$4.PE13; no longer IRIDIUM.19, U$1.A5
- net N$8: now also U$3.P$18, U$4.PB13; no longer GPS.2, U$1.B11
- net N$9: now also U$4.PD0, U$5.CTX; no longer U$1.A11, U$2.TXD
Routing:
- net GND: track 0.00 -> 268.0 mm, vias 0 -> 28
- net 3.3V: track 0.00 -> 179.6 mm, vias 0 -> 1
- net 5V_ICU: track 0.00 -> 124.7 mm, vias 0 -> 5
- net N$18: track 0.00 -> 78.7 mm
- net N$12: track 0.00 -> 68.2 mm
- net N$11: track 0.00 -> 66.7 mm, vias 0 -> 2
- net ON_OFF: track 0.00 -> 56.9 mm, vias 0 -> 3
- net N$9: track 0.00 -> 55.3 mm
- net N$10: track 0.00 -> 47.6 mm
- net N$17: track 0.00 -> 44.6 mm
- net N$13: track 0.00 -> 41.9 mm
- net N$16: track 0.00 -> 41.1 mm
- net N$8: track 0.00 -> 39.4 mm, vias 0 -> 1
- net N$15: track 0.00 -> 34.4 mm
- net N$2: track 0.00 -> 33.2 mm
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- added copper zone on layer 1, net GND
- added copper zone on layer 16, net GND
Other:
- board size 160 x 100 mm -> 85 x 100 mm

Commit message: Прихорошил плату ICU
Parts:
- moved JP1 22.9 mm to (65.1, 67.9)
- moved JP2 22.6 mm to (65.1, 63.3)
- moved ANT_IN 0.42 mm to (79.6, 50.3), turned to 0 degrees
Routing:
- net GND: track 268.0 -> 12.6 mm, vias 28 -> 47
- net 3.3V: track 179.6 -> 200.8 mm
- net 7.4V: track 18.5 -> 31.9 mm
- net N$12: track 68.2 -> 81.6 mm
- net N$8: track 39.4 -> 33.2 mm, vias 1 -> 0
- net N$9: track 55.3 -> 51.2 mm
- net 5V_ICU: track 124.7 -> 128.4 mm
- net N$5: track 23.6 -> 26.5 mm
- net N$10: track 47.6 -> 50.3 mm
- net N$11: track 66.7 -> 69.2 mm
- net ON_OFF: track 56.9 -> 58.1 mm
- net N$4: track 14.6 -> 13.8 mm
Other:
- outline, holes or cut-outs redrawn

Commit message: Скоро будут готовы ICU, SCU и CCU. Остались последние проверки
Connections:
- net 5V_ICU: now also U$4.5V_0
- net GND: now also U$4.GND_0, U$4.GND_1
Routing:
- net 5V_ICU: track 128.4 -> 131.4 mm
- net GND: track 12.6 -> 15.5 mm
