File: schematic/bumblebee/layerboards/out_board.brd (EAGLE design)
At the start: 92 x 25 mm, 15 parts, among them IC1 REG1117, X1 332-14, X2 332-08, X3 332-08, X4 332-06

Commit message: Все платы готовы и отправлены в резонит
Parts:
- added R1: 4k7, SparkFun-Resistors:AXIAL-0.3
- U$3: value LSMGY -> LSM303C; device bluepill:LSMGY -> bluepill:LSM303C
- moved U$3 1.60 mm to (10.6, 12.9)
Connections:
- net 3V3: now also R1.P$1
- net 5V: now also U$3.5V; no longer U$3.UCC
- net DQ: now also R1.P$2
- net MAG_CS: now also U$3.CSM; no longer U$3.CS
Routing:
- net SDA: track 33.2 -> 40.3 mm, vias 0 -> 1
- net SCL: track 34.9 -> 41.9 mm
- net DQ: track 19.9 -> 25.7 mm
- net 3V3: track 24.9 -> 29.1 mm
- net MAG_CS: track 36.6 -> 38.7 mm
- net 5V: track 51.0 -> 50.1 mm
Changed lines of the file:
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@@
 <attribute name="VALUE" x="21.52" y="7.4" size="1.27" layer="27"/>
-</element>
-<element name="U$3" library="bluepill" package="LSMGY" value="LSMGY" x="10.61" y="11.3" smashed="yes" rot="R180">
-<attribute name="VALUE" x="3.97" y="14.79" size="1.27" layer="27" rot="R270"/>
 </element>
 <element name="X1" library="con-garry" library_urn="urn:adsk.eagle:library:147" package="332-14" package3d_urn="urn:adsk.eagle:package:6814/1" value="332-14" x="55.68" y="15.64" smashed="yes" rot="R90"/>
@@
 <element name="X3" library="con-garry" library_urn="urn:adsk.eagle:library:147" package="332-08" package3d_urn="urn:adsk.eagle:package:6820/1" value="332-08" x="55.7" y="4.16" smashed="yes"/>
 <element name="X4" library="con-garry" library_urn="urn:adsk.eagle:library:147" package="332-06" package3d_urn="urn:adsk.eagle:package:6811/1" value="332-06" x="84.76" y="19.68" smashed="yes" rot="R90"/>
+<element name="U$3" library="bluepill" package="LSM303C" value="LSM303C" x="10.6" y="12.9" smashed="yes" rot="R180"/>
+<element name="R1" library="SparkFun-Resistors" package="AXIAL-0.3" value="4k7" x="24.4" y="1.9" smashed="yes" rot="R180">
+<attribute name="NAME" x="24.4" y="0.884" size="0.6096" layer="25" font="vector" ratio="20" rot="R180" align="bottom-center"/>
+<attribute name="PROD_ID" value=" " x="24.4" y="1.9" size="1.778" layer="27" rot="R180" display="off"/>
+<attribute name="VALUE" x="24.4" y="2.916" size="0.6096" layer="27" font="vector" ratio="20" rot="R180" align="top-center"/>
+</element>
 </elements>
 <signals>
@@
 <contactref element="U$2" pad="GND"/>
 <contactref element="U$1" pad="GND"/>
-<contactref element="U$3" pad="GND"/>
 <contactref element="X2" pad="8"/>
 <contactref element="X1" pad="8"/>
@@
 <wire x1="33" y1="10" x2="33.03" y2="10.03" width="0.2" layer="16"/>
 <wire x1="33.03" y1="10.03" x2="33.03" y2="12.37" width="0.2" layer="16"/>
+<contactref element="U$3" pad="GND"/>
 </signal>
 <signal name="3V3">
@@
 <wire x1="36.13" y1="1.94" x2="31.9" y2="6.17" width="0.2" layer="16"/>
 <wire x1="31.9" y1="6.17" x2="31.9" y2="11" width="0.2" layer="16"/>
+<contactref element="R1" pad="P$1"/>
+<wire x1="28.21" y1="1.9" x2="28.21" y2="3.25" width="0.2" layer="16"/>
+<wire x1="28.21" y1="3.25" x2="26.18" y2="5.28" width="0.2" layer="16"/>
 </signal>
 <signal name="5V">
 <contactref element="IC1" pad="3"/>
 <contactref element="C2" pad="1"/>
-<contactref element="U$3" pad="UCC"/>
 <contactref element="X2" pad="7"/>
 <wire x1="30.7186" y1="16.1004" x2="30.7186" y2="14.1914" width="0.2" layer="16"/>
@@
 <wire x1="30.73" y1="14.18" x2="23.25" y2="6.7" width="0.2" layer="16"/>
 <wire x1="23.25" y1="6.7" x2="21.4" y2="6.7" width="0.2" layer="16"/>
-<wire x1="21.4" y1="6.7" x2="17.11" y2="2.41" width="0.2" layer="16"/>
-<wire x1="17.11" y1="2.41" x2="15.69" y2="2.41" width="0.2" layer="16"/>
 <wire x1="49.97" y1="4.845075" x2="49.97" y2="5.714925" width="0.2" layer="16"/>
 <wire x1="48.92" y1="3.28" x2="48.92" y2="3.795075" width="0.2" layer="16"/>
@@
 <wire x1="31.9" y1="17.6" x2="30.7186" y2="16.4186" width="0.2" layer="16"/>
 <wire x1="30.7186" y1="16.4186" x2="30.7186" y2="16.1004" width="0.2" layer="16"/>
-<wire x1="42.043425" y1="7.1" x2="34.1039" y2="15.039525" width="0.2" layer="16"/>
-<wire x1="49.97" y1="5.714925" x2="48.584925" y2="7.1" width="0.2" layer="16"/>
-<wire x1="48.584925" y1="7.1" x2="42.043425" y2="7.1" width="0.2" layer="16"/>
+<contactref element="U$3" pad="5V"/>
+<wire x1="21.4" y1="6.7" x2="19.6" y2="4.9" width="0.2" layer="16"/>
+<wire x1="19.6" y1="4.9" x2="15.5" y2="4.9" width="0.2" layer="16"/>
+<wire x1="41.593425" y1="7.55" x2="34.1039" y2="15.039525" width="0.2" layer="16"/>
+<wire x1="48.134925" y1="7.55" x2="41.593425" y2="7.55" width="0.2" layer="16"/>
+<wire x1="49.97" y1="5.714925" x2="48.134925" y2="7.55" width="0.2" layer="16"/>
 </signal>
 <signal name="SWDIO_PCU">
@@
 </signal>
 <signal name="SDA">
+<contactref element="X2" pad="6"/>
 <contactref element="U$3" pad="SDA"/>
-<contactref element="X2" pad="6"/>
-<wire x1="46.92" y1="5.28" x2="46.404925" y2="5.28" width="0.2" layer="1"/>
-<wire x1="46.404925" y1="5.28" x2="45.354925" y2="6.33" width="0.2" layer="1"/>
-<wire x1="45.354925" y1="6.33" x2="27.7064" y2="6.33" width="0.2" layer="1"/>
-<wire x1="16.67" y1="9.05" x2="15.69" y2="10.03" width="0.2" layer="1"/>
-<wire x1="24.9864" y1="9.05" x2="16.67" y2="9.05" width="0.2" layer="1"/>
-<wire x1="27.7064" y1="6.33" x2="24.9864" y2="9.05" width="0.2" layer="1"/>
+<wire x1="46.92" y1="5.28" x2="45.1" y2="7.1" width="0.2" layer="16"/>
+<wire x1="45.1" y1="7.1" x2="40.37" y2="7.1" width="0.2" layer="16"/>
+<wire x1="40.37" y1="7.1" x2="37.7" y2="4.43" width="0.2" layer="16"/>
+<via x="37.7" y="4.43" extent="1-16" drill="0.5"/>
+<wire x1="28.57" y1="4.43" x2="37.7" y2="4.43" width="0.2" layer="1"/>
+<wire x1="15.5" y1="15.06" x2="17.76" y2="12.8" width="0.2" layer="1"/>
+<wire x1="17.76" y1="12.8" x2="17.76" y2="8.34" width="0.2" layer="1"/>
+<wire x1="25.7" y1="7.3" x2="28.57" y2="4.43" width="0.2" layer="1"/>
+<wire x1="17.76" y1="8.34" x2="18.8" y2="7.3" width="0.2" layer="1"/>
+<wire x1="18.8" y1="7.3" x2="25.7" y2="7.3" width="0.2" layer="1"/>
 </signal>
 <signal name="ADC_1">
@@
 </signal>
 <signal name="SCL">
-<contactref element="U$3" pad="SCL"/>
 <contactref element="X2" pad="5"/>
 <wire x1="46.92" y1="3.28" x2="46.404925" y2="3.28" width="0.2" layer="1"/>
-<wire x1="46.404925" y1="3.28" x2="44.064925" y2="0.94" width="0.2" layer="1"/>
-<wire x1="44.064925" y1="0.94" x2="22.24" y2="0.94" width="0.2" layer="1"/>
-<wire x1="22.24" y1="0.94" x2="15.69" y2="7.49" width="0.2" layer="1"/>
+<contactref element="U$3" pad="SCL"/>
+<wire x1="46.404925" y1="3.28" x2="43.624925" y2="0.5" width="0.2" layer="1"/>
+<wire x1="20.1" y1="0.5" x2="16.9" y2="3.7" width="0.2" layer="1"/>
+<wire x1="16.9" y1="3.7" x2="16.9" y2="11.12" width="0.2" layer="1"/>
+<wire x1="16.9" y1="11.12" x2="15.5" y2="12.52" width="0.2" layer="1"/>
+<wire x1="43.624925" y1="0.5" x2="20.1" y2="0.5" width="0.2" layer="1"/>
 </signal>
 <signal name="ADC_2">
@@
 </signal>
 <signal name="MAG_CS">
-<contactref element="U$3" pad="CS"/>
 <contactref element="X2" pad="2"/>
-<wire x1="42.92" y1="5.28" x2="28.12" y2="5.28" width="0.2" layer="1"/>
-<wire x1="24.8" y1="8.6" x2="15.2" y2="8.6" width="0.2" layer="1"/>
-<wire x1="15.2" y1="8.6" x2="14.2" y2="9.6" width="0.2" layer="1"/>
-<wire x1="14.2" y1="13.62" x2="15.69" y2="15.11" width="0.2" layer="1"/>
-<wire x1="28.12" y1="5.28" x2="24.8" y2="8.6" width="0.2" layer="1"/>
-<wire x1="14.2" y1="9.6" x2="14.2" y2="13.62" width="0.2" layer="1"/>
+<contactref element="U$3" pad="CSM"/>
+<wire x1="42.92" y1="5.28" x2="28.3564" y2="5.28" width="0.2" layer="1"/>
+<wire x1="25.8864" y1="7.75" x2="19.06" y2="7.75" width="0.2" layer="1"/>
+<wire x1="19.06" y1="7.75" x2="18.21" y2="8.6" width="0.2" layer="1"/>
+<wire x1="28.3564" y1="5.28" x2="25.8864" y2="7.75" width="0.2" layer="1"/>
+<wire x1="18.21" y1="8.6" x2="18.21" y2="12.99" width="0.2" layer="1"/>
+<wire x1="18.21" y1="12.99" x2="16.4" y2="14.8" width="0.2" layer="1"/>
+<wire x1="16.4" y1="14.8" x2="16.4" y2="19.24" width="0.2" layer="1"/>
+<wire x1="16.4" y1="19.24" x2="15.5" y2="20.14" width="0.2" layer="1"/>
 </signal>
 <signal name="DQ">
@@
 <wire x1="23.8" y1="5.28" x2="25.8" y2="3.28" width="0.2" layer="1"/>
 <wire x1="25.8" y1="3.28" x2="42.92" y2="3.28" width="0.2" layer="1"/>
+<contactref element="R1" pad="P$2"/>
+<wire x1="25.8" y1="3.28" x2="21.97" y2="3.28" width="0.2" layer="1"/>
+<wire x1="21.97" y1="3.28" x2="20.59" y2="1.9" width="0.2" layer="1"/>
 </signal>
 </signals>

Commit message: Все платы готовы и отправлены в Резонит
Other:
- board text added: "KeyHolder"
- board text added: "LSM303C"
- board text added: "Перед запуском убедитесь в исправности системы"
- board text added: "Спутникостроительный завод 2018-2019 OUT BOARD"
Changed lines of the file:
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@@
 <layer number="115" name="ReferenceISLANDS" color="7" fill="1" visible="no" active="no"/>
 <layer number="116" name="Patch_BOT" color="9" fill="4" visible="no" active="no"/>
+<layer number="117" name="BACKMAAT1" color="7" fill="1" visible="yes" active="yes"/>
 <layer number="118" name="Rect_Pads" color="7" fill="1" visible="no" active="no"/>
+<layer number="119" name="KAP_TEKEN" color="7" fill="1" visible="yes" active="yes"/>
+<layer number="120" name="KAP_MAAT1" color="7" fill="1" visible="yes" active="yes"/>
 <layer number="121" name="_tsilk" color="7" fill="1" visible="no" active="no"/>
 <layer number="122" name="_bsilk" color="7" fill="1" visible="no" active="no"/>
@@
 <layer number="128" name="_bValues" color="7" fill="1" visible="no" active="no"/>
 <layer number="129" name="Mask" color="7" fill="1" visible="no" active="no"/>
+<layer number="130" name="SMDSTROOK" color="7" fill="1" visible="yes" active="yes"/>
 <layer number="131" name="tAdjust" color="7" fill="1" visible="no" active="no"/>
 <layer number="132" name="bAdjust" color="7" fill="1" visible="no" active="no"/>
@@
 <text x="35.6" y="14.8" size="0.6" layer="22" rot="MR270">GND</text>
 <text x="29.5" y="12" size="0.6" layer="22" rot="MR0">GND</text>
-<text x="34.2" y="12.5" size="0.6" layer="22" rot="MR180">GND</text>
-<text x="17.3" y="4.7" size="0.6" layer="21">GND</text>
-<text x="17.5" y="2.3" size="0.6" layer="21">5V</text>
+<text x="34.2" y="12.1" size="0.6" layer="22" rot="MR180">GND</text>
+<text x="17.3" y="10.1" size="0.6" layer="21">GND</text>
+<text x="17.3" y="5" size="0.6" layer="21">5V</text>
 <text x="49" y="1.8" size="0.6" layer="22" rot="MR320">5V</text>
 <text x="46.9" y="6.3" size="0.6" layer="22" rot="MR140">SDA</text>
@@
 <text x="32.7" y="18" size="0.6" layer="22" rot="MR90">3V3</text>
 <text x="26" y="4.2" size="0.6" layer="22" rot="MR270">3V3</text>
+<text x="12.1" y="0.9" size="1" layer="21" rot="R90">Спутникостроительный завод
+2018-2019
+OUT BOARD</text>
+<text x="7.3" y="22.6" size="1" layer="21">LSM303C</text>
+<text x="66.2" y="1" size="1.2" layer="21" rot="R90">Перед запуском убедитесь
+в исправности системы</text>
+<text x="77.8" y="6.7" size="1" layer="21">KeyHolder</text>
 </plain>
 <attributes>
@@
 <elements>
 <element name="C1" library="SparkFun-Capacitors" package="0805" value="22uF" x="33.03" y="13.27" smashed="yes" rot="MR270">
-<attribute name="NAME" x="32.141" y="13.27" size="0.6096" layer="26" font="vector" ratio="20" rot="MR270" align="bottom-center"/>
 <attribute name="PROD_ID" value="CAP-08402" x="123.2" y="-26.1" size="1.778" layer="28" rot="MR270" display="off"/>
 <attribute name="VALUE" x="33.919" y="13.27" size="0.6096" layer="28" font="vector" ratio="20" rot="MR270" align="top-center"/>
 </element>
 <element name="C2" library="SparkFun-Capacitors" package="0805" value="10uF" x="30.73" y="13.28" smashed="yes" rot="MR270">
-<attribute name="NAME" x="29.841" y="13.28" size="0.6096" layer="26" font="vector" ratio="20" rot="MR270" align="bottom-center"/>
 <attribute name="PROD_ID" value="CAP-14260" x="120.9" y="-29.9" size="1.778" layer="28" rot="MR270" display="off"/>
 <attribute name="VALUE" x="31.619" y="13.28" size="0.6096" layer="28" font="vector" ratio="20" rot="MR270" align="top-center"/>
@@
 </element>
 <element name="U$2" library="bluepill" package="TEMP" value="TEMP" x="23.8" y="4.78" smashed="yes" rot="R270">
-<attribute name="NAME" x="27.3" y="6.28" size="1.27" layer="25" rot="R270"/>
 <attribute name="VALUE" x="21.52" y="7.4" size="1.27" layer="27"/>
 </element>
@@
 <element name="U$3" library="bluepill" package="LSM303C" value="LSM303C" x="10.6" y="12.9" smashed="yes" rot="R180"/>
 <element name="R1" library="SparkFun-Resistors" package="AXIAL-0.3" value="4k7" x="24.4" y="1.9" smashed="yes" rot="R180">
-<attribute name="NAME" x="24.4" y="0.884" size="0.6096" layer="25" font="vector" ratio="20" rot="R180" align="bottom-center"/>
 <attribute name="PROD_ID" value=" " x="24.4" y="1.9" size="1.778" layer="27" rot="R180" display="off"/>
-<attribute name="VALUE" x="24.4" y="2.916" size="0.6096" layer="27" font="vector" ratio="20" rot="R180" align="top-center"/>
+<attribute name="VALUE" x="24.4" y="1.716" size="0.6096" layer="27" font="vector" ratio="20" rot="R180" align="top-center"/>
 </element>
 </elements>
@@
 <wire x1="30.7186" y1="14.1914" x2="30.73" y2="14.18" width="0.2" layer="16"/>
 <wire x1="30.73" y1="14.18" x2="23.25" y2="6.7" width="0.2" layer="16"/>
-<wire x1="23.25" y1="6.7" x2="21.4" y2="6.7" width="0.2" layer="16"/>
+<wire x1="23.25" y1="6.7" x2="21.1" y2="6.7" width="0.2" layer="16"/>
 <wire x1="49.97" y1="4.845075" x2="49.97" y2="5.714925" width="0.2" layer="16"/>
 <wire x1="48.92" y1="3.28" x2="48.92" y2="3.795075" width="0.2" layer="16"/>
@@
 <wire x1="30.7186" y1="16.4186" x2="30.7186" y2="16.1004" width="0.2" layer="16"/>
 <contactref element="U$3" pad="5V"/>
-<wire x1="21.4" y1="6.7" x2="19.6" y2="4.9" width="0.2" layer="16"/>
-<wire x1="19.6" y1="4.9" x2="15.5" y2="4.9" width="0.2" layer="16"/>
+<wire x1="21.1" y1="6.7" x2="19.7" y2="5.3" width="0.2" layer="16"/>
+<wire x1="19.7" y1="5.3" x2="19.6981" y2="5.28" width="0.2" layer="16"/>
+<wire x1="19.6981" y1="5.28" x2="15.6" y2="5.28" width="0.2" layer="16"/>
 <wire x1="41.593425" y1="7.55" x2="34.1039" y2="15.039525" width="0.2" layer="16"/>
 <wire x1="48.134925" y1="7.55" x2="41.593425" y2="7.55" width="0.2" layer="16"/>
@@
 <via x="37.7" y="4.43" extent="1-16" drill="0.5"/>
 <wire x1="28.57" y1="4.43" x2="37.7" y2="4.43" width="0.2" layer="1"/>
-<wire x1="15.5" y1="15.06" x2="17.76" y2="12.8" width="0.2" layer="1"/>
+<wire x1="15.6" y1="15.44" x2="17.76" y2="12.8" width="0.2" layer="1"/>
 <wire x1="17.76" y1="12.8" x2="17.76" y2="8.34" width="0.2" layer="1"/>
 <wire x1="25.7" y1="7.3" x2="28.57" y2="4.43" width="0.2" layer="1"/>
@@
 <wire x1="20.1" y1="0.5" x2="16.9" y2="3.7" width="0.2" layer="1"/>
 <wire x1="16.9" y1="3.7" x2="16.9" y2="11.12" width="0.2" layer="1"/>
-<wire x1="16.9" y1="11.12" x2="15.5" y2="12.52" width="0.2" layer="1"/>
+<wire x1="16.9" y1="11.12" x2="15.6" y2="12.9" width="0.2" layer="1"/>
 <wire x1="43.624925" y1="0.5" x2="20.1" y2="0.5" width="0.2" layer="1"/>
 </signal>
@@
 <wire x1="19.06" y1="7.75" x2="18.21" y2="8.6" width="0.2" layer="1"/>
 <wire x1="28.3564" y1="5.28" x2="25.8864" y2="7.75" width="0.2" layer="1"/>
-<wire x1="18.21" y1="8.6" x2="18.21" y2="12.99" width="0.2" layer="1"/>
-<wire x1="18.21" y1="12.99" x2="16.4" y2="14.8" width="0.2" layer="1"/>
-<wire x1="16.4" y1="14.8" x2="16.4" y2="19.24" width="0.2" layer="1"/>
-<wire x1="16.4" y1="19.24" x2="15.5" y2="20.14" width="0.2" layer="1"/>
+<wire x1="18.21" y1="8.6" x2="18.21" y2="16.344" width="0.2" layer="1"/>
+<wire x1="18.21" y1="16.344" x2="15.6" y2="20.52" width="0.2" layer="1"/>
 </signal>
 <signal name="DQ">
@@
 </drawing>
 <compatibility>
+<note version="6.3" minversion="6.2.2" severity="warning">
+Since Version 6.2.2 text objects can contain more than one line,
+which will not be processed correctly with this version.
+</note>
 <note version="8.2" severity="warning">
 Since Version 8.2, EAGLE supports online libraries. The ids
