File: schematic/bumblebee/devboards/devboards-panel.brd (EAGLE design)
At the start: 98 x 52 mm, 13 parts, among them J1 U.FL-R-SMT(01)

Commit message: Нашелся первый косяк на платах
Connections:
- new net GND2: J1.1, J1.2
