File: schematic/bumblebee/devboards/iridium-by-262-breakout.brd (EAGLE design)
At the start: 36 x 30 mm, 2 parts, among them J1 U.FL-R-SMT(01)

Commit message: Нашелся первый косяк на платах
Connections:
- new net GND: J1.1, J1.2
Changed lines of the file:
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@@
 <via x="33" y="23" extent="1-16" drill="0.5"/>
 <via x="7" y="2" extent="1-16" drill="0.5"/>
+<contactref element="J1" pad="1"/>
+<contactref element="J1" pad="2"/>
 </signal>
 </signals>
